File: modules/AC_PowerController/AC_PowerController.kicad_pcb (KiCad board)
At the start: 2 copper layers, 34 parts, among them J5 114020164, Q1 IRF640, Q2 IRF640, U1 AMC23C10, U2 TPSI3050QDWZRQ1

Commit message: update
Parts:
- moved J101 22.9 mm to (181.8, 50.0)
- moved H108 20.1 mm to (131.9, 56.6)
- moved H106 18.6 mm to (131.9, 50.6)
- moved Q101 18.3 mm to (119.5, 50.6)
- moved Q102 17.8 mm to (119.5, 76.2)
- moved C106 17.4 mm to (164.8, 54.1), turned to -90 degrees
- moved H107 16.8 mm to (127.7, 53.6)
- moved H110 16.1 mm to (131.9, 62.6)
- moved H105 15.0 mm to (127.7, 47.6)
- moved C108 14.0 mm to (172.2, 47.9)
- moved H101 13.6 mm to (127.7, 65.6)
- moved H109 13.2 mm to (127.7, 59.6)
- moved H102 12.5 mm to (131.9, 68.6)
- moved H104 11.1 mm to (131.9, 74.6)
- moved R104 10.7 mm to (170.8, 66.1)
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- renumbered C1 to C101, C2 to C102, C3 to C103, C4 to C104, C5 to C105, C6 to C106, C7 to C107, C8 to C108, C9 to C109, D1 to D101, D2 to D102, H6 to H101, H7 to H102, H8 to H103, H9 to H104, H2 to H105, H3 to H106, H4 to H107, H5 to H108, H10 to H109, H11 to H110, J5 to J101, JP1 to JP101, JP2 to JP102, JP3 to JP103, JP4 to JP104, Q1 to Q101, Q2 to Q102, R1 to R101, R2 to R102, R3 to R103, R4 to R104, U1 to U101, U2 to U102
Routing:
- net VSSS: track 0.00 -> 72.2 mm
- net VDD1: track 0.00 -> 49.4 mm
- net Net-(Q101-G): track 0.00 -> 46.3 mm, vias 0 -> 3
- net VDD: track 0.00 -> 35.5 mm
- net /AC_N: track 0.00 -> 29.1 mm
- net Net-(Q101-D): track 0.00 -> 20.4 mm
- net Net-(D101-A): track 0.00 -> 14.8 mm
- net /ZC2: track 0.00 -> 10.4 mm
- net /VDDM: track 0.00 -> 8.44 mm
- net Net-(JP101-A): track 0.00 -> 6.96 mm
- net Net-(U102-VDDH): track 0.00 -> 6.71 mm
- net Net-(H102-Pad1): track 0.00 -> 6.00 mm
- net Net-(H101-Pad1): track 0.00 -> 6.00 mm
- net /ZC1: track 0.00 -> 5.64 mm
- net Net-(H106-Pad1): track 0.00 -> 5.49 mm
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