File: modules/AC_PowerController/AC_PowerController.kicad_sch (KiCad schematic)
At the start: 34 parts, among them J5 114020164, Q1 IRF640, Q2 IRF640, U1 AMC23C10, U2 TPSI3050QDWZRQ1

Commit message: update
Parts:
- H101: renamed from H6; now not fitted
- H102: renamed from H7; now not fitted
- H103: renamed from H8; now not fitted
- H104: renamed from H9; now not fitted
- H105: renamed from H2; now not fitted
- H106: renamed from H3; now not fitted
- H107: renamed from H4; now not fitted
- H108: renamed from H5; now not fitted
- H109: renamed from H10; now not fitted
- H110: renamed from H11; now not fitted
- renumbered C1 to C101, C2 to C102, C3 to C103, C4 to C104, C5 to C105, C6 to C106, C7 to C107, C8 to C108, C9 to C109, D1 to D101, D2 to D102, J5 to J101, JP1 to JP101, JP2 to JP102, JP3 to JP103, JP4 to JP104, Q1 to Q101, Q2 to Q102, R1 to R101, R2 to R102, R3 to R103, R4 to R104, U1 to U101, U2 to U102
