File: modules/I2C_TempSenser/I2C_TempSenser.kicad_sch (KiCad schematic)
At the start: 11 parts, among them J101 SolderPAD, U101 TPS7A2033DQN, U102 PCA9306YZTR, U103 TMP119AIYBGR

Commit message: update
Parts:
- removed C103, C105, C107: 104C10, Capacitor_SMD:C_0201_0603Metric, symbol Device:C_Small
- removed J101: SolderPAD, symbol Connector:Conn_01x04_Pin
- removed U102: PCA9306YZTR, Package_BGA:Texas_DSBGA-8_0.9x1.9mm_Layout2x4_P0.5mm, symbol Interface:PCA9306
- added FB101: BLM03BX182SN1D, Inductor_SMD:L_0201_0603Metric, symbol Device:FerriteBead_Small
- added R101, R103, R104: 0, Resistor_SMD:R_0201_0603Metric, symbol Device:R_Small
- added R102, R105: 333C1S20, Resistor_SMD:R_0201_0603Metric, symbol Device:R_Small
- added TP101, TP102, TP103, TP104, TP105: P5V, 0_Pad:Oval_Pad_1.0x4.0mm, symbol Connector:TestPoint
- added U102: P82B715DR, Package_SO:SOIC-8_3.9x4.9mm_P1.27mm, symbol 00_Make:P82B715
- C101: Manufacturer Product Number (none) -> GRM033R61A105ME44D
- C102, C104: value 104C10 -> 104C6P3; Manufacturer Product Number (none) -> GRM033R60J104KE19D
- C103: renamed from C106; value 104C10 -> 104C6P3; Manufacturer Product Number (none) -> GRM033R60J104KE19D
Connections:
- net +3.3V: now also C104.1, R103.2
- net +5V: now also FB101.2, R102.1, R103.1, R105.1, U102.5 (VCC); no longer C104.1
- net GND: now also TP102.1, TP105.1, U102.4 (GND)
- net SCL1: now also U103.A2 (SCL), R104.2, R105.2, U102.7 (Ly)
- net SCL2: now also R104.1, TP103.1, U102.6 (Sy); no longer U103.A2 (SCL)
- net SDA1: now also U103.A1 (SDA), R101.2, R102.2, U102.2 (Lx)
- net SDA2: now also R101.1, TP104.1, U102.3 (Sx); no longer U103.A1 (SDA)
- new net: FB101.1, TP101.1
Other:
- moved on the sheet: C103, U101, U103
